File: bbq20kbd_connector.kicad_sch (KiCad schematic)
At the start: 31 parts, among them J8 BBQ20KBD, J9 BBQ20KBD GPIOs, Q1 BSS138, Q2 BSS138, Q3 BSS138, Q4 BSS138, Q5 BSS138, Q6 BSS138

Commit message: Begin PCB
Parts:
- removed J9: BBQ20KBD GPIOs, Connector_IDC:IDC-Header_2x20_P2.54mm_Vertical, symbol Connector_Generic:Conn_02x20_Top_Bottom
- removed JP1: P24, TestPoint:TestPoint_2Pads_Pitch2.54mm_Drill0.8mm, symbol Jumper:Jumper_2_Open
- removed JP10: LEDK, TestPoint:TestPoint_2Pads_Pitch2.54mm_Drill0.8mm, symbol Jumper:Jumper_2_Open
- removed JP11: P22, TestPoint:TestPoint_2Pads_Pitch2.54mm_Drill0.8mm, symbol Jumper:Jumper_2_Open
- removed JP12: P01, TestPoint:TestPoint_2Pads_Pitch2.54mm_Drill0.8mm, symbol Jumper:Jumper_2_Open
- removed JP2: P08, TestPoint:TestPoint_2Pads_Pitch2.54mm_Drill0.8mm, symbol Jumper:Jumper_2_Open
- removed JP3: P10, TestPoint:TestPoint_2Pads_Pitch2.54mm_Drill0.8mm, symbol Jumper:Jumper_2_Open
- removed JP4: LEDA, TestPoint:TestPoint_2Pads_Pitch2.54mm_Drill0.8mm, symbol Jumper:Jumper_2_Open
- removed JP5: TP_MOTION, TestPoint:TestPoint_2Pads_Pitch2.54mm_Drill0.8mm, symbol Jumper:Jumper_2_Open
- removed JP6: TP_SCL, TestPoint:TestPoint_2Pads_Pitch2.54mm_Drill0.8mm, symbol Jumper:Jumper_2_Open
- removed JP7: TP_SDA, TestPoint:TestPoint_2Pads_Pitch2.54mm_Drill0.8mm, symbol Jumper:Jumper_2_Open
- removed JP8: TP_RESET, TestPoint:TestPoint_2Pads_Pitch2.54mm_Drill0.8mm, symbol Jumper:Jumper_2_Open
- removed JP9: TP_SHUTDOWN, TestPoint:TestPoint_2Pads_Pitch2.54mm_Drill0.8mm, symbol Jumper:Jumper_2_Open
- added C3, C4, C5, C6: 1uF, Capacitor_SMD:C_0603_1608Metric, symbol Device:C
- added U2: TPS7A2018PDBVR, Package_TO_SOT_SMD:SOT-23-5, symbol Regulator_Linear:TPS73618DBV
- added U3: TPS7A2028PDBVR, Package_TO_SOT_SMD:SOT-23-5, symbol Regulator_Linear:TPS73618DBV
- J8: footprint (none) -> Connector_Hirose:Hirose_BM20B0.8-40DS-0.4V
Connections:
- net LEDA is gone; now on net +3V3: J8.34 (VDD_BKL)
- net LEDK is gone; now on net BKL: J8.33 (N.C)
- net P01 is gone; now on net GND: J8.1 (GND)
- net P08 is gone; now on net +2V8: J8.8 (VDD_KBD)
- net P10 is gone; now on net +1V8: J8.10 (VDD_TP)
- net P22 is gone; now on net GND: J8.22 (AGND)
- net P24 is gone; now on net +3V3: J8.24 (VDD_MIC)
- net +1V8: now also C4.1, U2.5 (OUT)
- net +2V8: now also C6.1, U3.5 (OUT)
- net +3V3: now also C3.1, C5.2, U2.1 (IN), U2.3 (EN), U3.1 (IN), U3.3 (EN)
- net BKL: now also Q6.3 (D)
- net GND: now also C3.2, C4.2, C5.1, C6.2, U2.2 (GND), U3.2 (GND)
- net TP_MOTION_1V8: now also Q4.2 (S), R8.1
- net TP_RESET_1V8: now also Q5.2 (S), R10.1
- net TP_SCL_1V8: now also Q2.2 (S), R4.1
- net TP_SDA_1V8: now also Q3.2 (S), R6.1
- net TP_SHUTDOWN_1V8: now also Q1.2 (S), R2.1
- net COL0 renamed KBD_COL0
- net COL1 renamed KBD_COL1
- net COL2 renamed KBD_COL2
- net COL3 renamed KBD_COL3
- net COL4 renamed KBD_COL4
- net COL5 renamed KBD_COL5
- net COL6 renamed KBD_COL6
- net P07: no longer names the net of J8.7 (N.C)
- net P09: no longer names the net of J8.9 (N.C)
- net P11: no longer names the net of J8.11 (N.C)
- net P19: no longer names the net of J8.19 (N.C)
- net P20: no longer names the net of J8.20 (N.C)
- net P21: no longer names the net of J8.21 (N.C)
- net P25: no longer names the net of J8.25 (N.C)
- net P35: no longer names the net of J8.35 (N.C)
- net P36: no longer names the net of J8.36 (N.C)
- net P37: no longer names the net of J8.37 (N.C)
- net P38: no longer names the net of J8.38 (N.C)
- net P39: no longer names the net of J8.39 (N.C)
- net P40: no longer names the net of J8.40 (N.C)
- net ROW0 renamed KBD_ROW0
- net ROW1 renamed KBD_ROW1
- net ROW2 renamed KBD_ROW2
- net ROW3 renamed KBD_ROW3
- net ROW4 renamed KBD_ROW4
- net ROW5 renamed KBD_ROW5
- net ROW6 renamed KBD_ROW6
- no-connect marks 0 -> 2
Other:
- moved on the sheet: Q1, Q2, Q3, Q4, Q5, Q6, R1, R10, R11, R2, R3, R4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

Commit message: Version 1
Parts:
- renumbered Q3 to Q2, Q2 to Q3, R5 to R3, R6 to R4, R3 to R5, R4 to R6
Connections:
- net BKL: no longer Q6.1 (G), R11.2
- new net KBD_BKL: Q6.1 (G), R11.2
Other:
- moved on the sheet: C3, C4, C5, C6, J8, Q1, Q2, Q3, Q4, Q5, Q6, R1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
