File: gp-bbq20kbd-breakout-board.kicad_pcb (KiCad board)
At the start: 4 copper layers, 100 x 75 mm, 42 parts, among them J1 PWR, J2 KEYBOARD, J3 MOTION, J4 MIC, J5 BKL, J8 BBQ20KBD, Q1 BSS138, Q2 BSS138, Q3 BSS138, Q4 BSS138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

Commit message: Version 1
Parts:
- J2: footprint Connector_PinHeader_2.54mm:PinHeader_2x07_P2.54mm_Vertical -> Connector_PinHeader_2.54mm:PinHeader_1x14_P2.54mm_Vertical
- moved J2 66.1 mm to (120.5, 52.0), turned to 90 degrees
- moved D1 25.0 mm to (175.0, 55.0)
- moved J3 18.0 mm to (187.9, 74.9)
- moved J5 17.2 mm to (188.0, 97.0)
- moved J4 7.14 mm to (188.0, 102.0)
- moved R11 6.08 mm to (175.0, 96.0), turned to -90 degrees
- moved C5 5.91 mm to (177.5, 109.9), turned to 90 degrees
- moved C6 5.91 mm to (170.5, 109.9)
- moved U3 5.91 mm to (174.0, 109.9)
- moved TP3 5.00 mm to (170.0, 115.0)
- moved J1 3.23 mm to (188.0, 61.5)
- moved TP5 2.00 mm to (170.0, 55.0)
- moved Q6 1.00 mm to (172.0, 96.0), turned to 180 degrees
- moved C4 0.50 mm to (171.0, 66.0)
- moved C3 0.50 mm to (177.0, 66.0)
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Connections:
- J2 pad 10: /KBD_ROW4 -> /KBD_ROW2
- J2 pad 11: /KBD_COL5 -> /KBD_ROW3
- J2 pad 12: /KBD_ROW5 -> /KBD_ROW4
- J2 pad 13: /KBD_COL6 -> /KBD_ROW5
- J2 pad 2: /KBD_ROW0 -> /KBD_COL1
- J2 pad 3: /KBD_COL1 -> /KBD_COL2
- J2 pad 4: /KBD_ROW1 -> /KBD_COL3
- J2 pad 5: /KBD_COL2 -> /KBD_COL4
- J2 pad 6: /KBD_ROW2 -> /KBD_COL5
- J2 pad 7: /KBD_COL3 -> /KBD_COL6
- J2 pad 8: /KBD_ROW3 -> /KBD_ROW0
- J2 pad 9: /KBD_COL4 -> /KBD_ROW1
- J3 pad 1: /TP_MOTION -> /TP_SHUTDOWN
- J3 pad 2: /TP_SCL -> /TP_SDA
- J3 pad 3: /TP_SDA -> /TP_SCL
- J3 pad 4: /TP_SHUTDOWN -> /TP_MOTION
- J5 pad 1: /BKL -> /KBD_BKL
- J8 pad 33: /BKL -> /bbq20kbd_connector/BKL
- Q1 pad 3: /TP_RESET -> /TP_SHUTDOWN
- Q2 pad 2: /bbq20kbd_connector/TP_SCL_1V8 -> /bbq20kbd_connector/TP_SDA_1V8
- Q2 pad 3: /TP_SCL -> /TP_SDA
- Q3 pad 2: /bbq20kbd_connector/TP_SDA_1V8 -> /bbq20kbd_connector/TP_SCL_1V8
- Q3 pad 3: /TP_SDA -> /TP_SCL
- Q5 pad 3: /TP_SHUTDOWN -> /TP_RESET
- Q6 pad 1: /BKL -> /KBD_BKL
- Q6 pad 3: /BKL -> /bbq20kbd_connector/BKL
- R1 pad 1: /TP_RESET -> /TP_SHUTDOWN
- R11 pad 2: /BKL -> /KBD_BKL
- R3 pad 1: /TP_SCL -> /TP_SDA
- R4 pad 1: /bbq20kbd_connector/TP_SCL_1V8 -> /bbq20kbd_connector/TP_SDA_1V8
- R5 pad 1: /TP_SDA -> /TP_SCL
- R6 pad 1: /bbq20kbd_connector/TP_SDA_1V8 -> /bbq20kbd_connector/TP_SCL_1V8
- R9 pad 1: /TP_SHUTDOWN -> /TP_RESET
Routing:
- net /MIC: track 0.00 -> 96.0 mm, vias 0 -> 1
- net /bbq20kbd_connector/TP_RESET_1V8: track 0.00 -> 78.2 mm, vias 0 -> 2
- net /bbq20kbd_connector/BKL: track 0.00 -> 77.6 mm, vias 0 -> 2
- net /bbq20kbd_connector/TP_MOTION_1V8: track 0.00 -> 74.9 mm, vias 0 -> 2
- net /bbq20kbd_connector/TP_SHUTDOWN_1V8: track 0.00 -> 74.2 mm, vias 0 -> 2
- net /bbq20kbd_connector/TP_SCL_1V8: track 0.00 -> 73.6 mm, vias 0 -> 2
- net /bbq20kbd_connector/TP_SDA_1V8: track 0.00 -> 72.9 mm, vias 0 -> 2
- net GND: track 0.00 -> 60.4 mm, vias 0 -> 5
- net /KBD_ROW6: track 0.00 -> 59.9 mm
- net +3V3: track 1.82 -> 61.3 mm, vias 0 -> 10
- net /KBD_ROW5: track 0.00 -> 57.2 mm
- net /KBD_ROW4: track 0.00 -> 54.5 mm
- net /KBD_ROW3: track 0.00 -> 51.7 mm
- net /KBD_ROW2: track 0.00 -> 49.0 mm
- net /KBD_ROW1: track 0.00 -> 46.3 mm
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- removed copper zone on In2.Cu, net +5V
